Commit message: From RPi

File: toto2_desc/models/toto2.xacro (robot description, xacro)
@@ -67,16 +67,4 @@
     </collision>
   </link>
-  <joint name="left_wheel_joint" type="continuous">
-    <origin xyz=" 0.0 0.1195 0.0499" rpy="0 0 -1.57079633"/>
-    <parent link="base_link"/>
-    <child link="left_wheel_1"/>
-    <axis xyz="-1.0 0.0 0.0"/>
-  </joint>
-  <joint name="right_wheel_joint" type="continuous">
-    <origin xyz="0.0 -0.1195 0.0499" rpy="0 0 -1.57079633"/>
-    <parent link="base_link"/>
-    <child link="right_wheel_1"/>
-    <axis xyz="-1.0 0.0 0.0"/>
-  </joint>
   <!-- THE FOLLOWING ARE SENSOR DESCRIPTORS-->
   <!-- LIDAR -->
@@ -101,9 +89,4 @@
     </collision>
   </link>
-  <joint name="lidar_joint" type="fixed">
-    <parent link="base_link"/>
-    <child link="lidar_1"/>
-    <origin xyz="0.1 0.0 0.17" rpy="0 0 0"/>
-  </joint>
   <!-- CAMERA -->
   <link name="camera_link1_1">
@@ -115,4 +98,10 @@
   <link name="imu_link">
   </link>
+  <!-- Joints -->
+  <joint name="lidar_joint" type="fixed">
+    <parent link="base_link"/>
+    <child link="lidar_1"/>
+    <origin xyz="0.1 0.0 0.17" rpy="0 0 3.14"/>
+  </joint>
   <joint name="base" type="fixed">
     <parent link="base_footprint"/>
@@ -144,3 +133,25 @@
     <origin xyz="0.020 0.01 0.015" rpy="0 0 0" />
   </joint>
+  <joint name="left_wheel_joint" type="fixed">
+    <origin xyz=" 0.0 0.1195 0.0499" rpy="0 0 -1.57079633"/>
+    <parent link="base_link"/>
+    <child link="left_wheel_1"/>
+  </joint>
+  <joint name="right_wheel_joint" type="fixed">
+    <origin xyz="0.0 -0.1195 0.0499" rpy="0 0 -1.57079633"/>
+    <parent link="base_link"/>
+    <child link="right_wheel_1"/>
+  </joint>
+  <!-- <joint name="left_wheel_joint" type="continuous">
+    <origin xyz=" 0.0 0.1195 0.0499" rpy="0 0 -1.57079633"/>
+    <parent link="base_link"/>
+    <child link="left_wheel_1"/>
+    <axis xyz="-1.0 0.0 0.0"/>
+  </joint>
+  <joint name="right_wheel_joint" type="continuous">
+    <origin xyz="0.0 -0.1195 0.0499" rpy="0 0 -1.57079633"/>
+    <parent link="base_link"/>
+    <child link="right_wheel_1"/>
+    <axis xyz="-1.0 0.0 0.0"/>
+  </joint> -->
 </robot>

Commit message: nav2 stack implemented without tuning

File: toto2_desc/models/toto2.xacro (robot description, xacro)
@@ -18,5 +18,5 @@
         <mesh filename="package://toto2_description/meshes/base_link.stl" scale="0.001 0.001 0.001"/>
       </geometry>
-      <material name="silver"/>
+      <!-- <material name="silver"/> -->
     </visual>
     <collision>
@@ -38,5 +38,5 @@
         <mesh filename="package://toto2_description/meshes/right_wheel_1.stl" scale="0.001 0.001 0.001"/>
       </geometry>
-      <material name="silver"/>
+      <!-- <material name="silver"/> -->
     </visual>
     <collision>
@@ -58,5 +58,5 @@
         <mesh filename="package://toto2_description/meshes/left_wheel_1.stl" scale="0.001 0.001 0.001"/>
       </geometry>
-      <material name="silver"/>
+      <!-- <material name="silver"/> -->
     </visual>
     <collision>
@@ -80,5 +80,5 @@
         <mesh filename="package://toto2_description/meshes/lidar_1.stl" scale="0.001 0.001 0.001"/>
       </geometry>
-      <material name="silver"/>
+      <!-- <material name="silver"/> -->
     </visual>
     <collision>

Commit message: Navigation working

File: toto2_desc/models/toto2.xacro (robot description, xacro)
@@ -131,5 +131,5 @@
     <parent link="camera_link2_1"/>
     <child link="camera_1"/>
-    <origin xyz="0.020 0.01 0.015" rpy="0 0 0" />
+    <origin xyz="0.020 0.01 0.015" rpy="-1.57079632679 0 -1.57079632679" />
   </joint>
   <joint name="left_wheel_joint" type="fixed">

Commit message: minor changes

File: toto2_desc/models/toto2.xacro (robot description, xacro)
@@ -116,5 +116,5 @@
     <axis xyz="0.0 0.0 1.0" />
   </joint>
-  <joint name="camera_joint_1" type="fixed">
+  <!-- <joint name="camera_joint_1" type="fixed">
     <parent link="base_link"/>
     <child link="camera_link1_1"/>
@@ -123,4 +123,16 @@
   </joint>
   <joint name="camera_joint_2" type="fixed">
+    <parent link="camera_link1_1"/>
+    <child link="camera_link2_1"/>
+    <origin xyz="0.03 0.0 0.042" rpy="0 0 0" />
+    <axis xyz="0.0 1.0 0.0" />
+  </joint> -->
+  <joint name="camera_joint_1" type="continuous">
+    <parent link="base_link"/>
+    <child link="camera_link1_1"/>
+    <origin xyz="0.16 0.0 0.2795" rpy="0 0 0" />
+    <axis xyz="0.0 0.0 1.0" />
+  </joint>
+  <joint name="camera_joint_2" type="continuous">
     <parent link="camera_link1_1"/>
     <child link="camera_link2_1"/>

Commit message: Changed params to integrate sharp sensor with nav2 stack

File: toto2_desc/models/toto2.xacro (robot description, xacro)
@@ -96,5 +96,11 @@
   <link name="camera_1">
   </link>
+  <!-- IMU -->
   <link name="imu_link">
+  </link>
+  <!-- SHARP SENSOR -->
+  <link name="left_sharp">
+  </link>
+  <link name="right_sharp">
   </link>
   <!-- Joints -->
@@ -103,4 +109,14 @@
     <child link="lidar_1"/>
     <origin xyz="0.1 0.0 0.17" rpy="0 0 3.14"/>
+  </joint>
+  <joint name="left_sharp_joint" type="fixed">
+    <parent link="base_link"/>
+    <child link="left_sharp"/>
+    <origin xyz="0.187 0.14 0.0" rpy="0 0.7853981 0"/>
+  </joint>
+  <joint name="right_sharp_joint" type="fixed">
+    <parent link="base_link"/>
+    <child link="right_sharp"/>
+    <origin xyz="0.187 -0.14 0.0" rpy="0 0.7853981 0"/>
   </joint>
   <joint name="base" type="fixed">
@@ -132,5 +148,5 @@
     <child link="camera_link1_1"/>
     <origin xyz="0.16 0.0 0.2795" rpy="0 0 0" />
-    <axis xyz="0.0 0.0 1.0" />
+    <axis xyz="0.0 0.0 -1.0" />
   </joint>
   <joint name="camera_joint_2" type="continuous">

Commit message: Updates

File: toto2_desc/models/toto2.xacro (robot description, xacro)
@@ -90,13 +90,13 @@
   </link>
   <!-- CAMERA -->
-  <link name="camera_link1_1">
+  <link name="camera_link1">
   </link>
-  <link name="camera_link2_1">
+  <link name="camera_link2">
   </link>
   <link name="camera_1">
   </link>
   <!-- IMU -->
-  <link name="imu_link">
-  </link>
+  <!-- <link name="imu_link">
+  </link> -->
   <!-- SHARP SENSOR -->
   <link name="left_sharp">
@@ -113,32 +113,32 @@
     <parent link="base_link"/>
     <child link="left_sharp"/>
-    <origin xyz="0.187 0.14 0.0" rpy="0 0.7853981 0"/>
+    <origin xyz="0.187 0.14 0.08" rpy="0 0.7853981 0"/>
   </joint>
   <joint name="right_sharp_joint" type="fixed">
     <parent link="base_link"/>
     <child link="right_sharp"/>
-    <origin xyz="0.187 -0.14 0.0" rpy="0 0.7853981 0"/>
+    <origin xyz="0.187 -0.14 0.08" rpy="0 0.7853981 0"/>
   </joint>
   <joint name="base" type="fixed">
     <parent link="base_footprint"/>
     <child link="base_link"/>
-    <origin xyz="0.0 0.0 0.1" rpy="0 0 0" />
+    <origin xyz="0.0 0.0 0.0" rpy="0 0 0" />
     <axis xyz="0.0 0.0 1.0" />
   </joint>
-  <joint name="imu_joint" type="fixed">
+  <!-- <joint name="imu_joint" type="fixed">
     <parent link="base_link"/>
     <child link="imu_link"/>
     <origin xyz="0.0 0.0 0.17" rpy="0 0 0" />
     <axis xyz="0.0 0.0 1.0" />
-  </joint>
+  </joint> -->
   <!-- <joint name="camera_joint_1" type="fixed">
     <parent link="base_link"/>
-    <child link="camera_link1_1"/>
+    <child link="camera_link1"/>
     <origin xyz="0.16 0.0 0.2795" rpy="0 0 0" />
     <axis xyz="0.0 0.0 1.0" />
   </joint>
   <joint name="camera_joint_2" type="fixed">
-    <parent link="camera_link1_1"/>
-    <child link="camera_link2_1"/>
+    <parent link="camera_link1"/>
+    <child link="camera_link2"/>
     <origin xyz="0.03 0.0 0.042" rpy="0 0 0" />
     <axis xyz="0.0 1.0 0.0" />
@@ -146,16 +146,16 @@
   <joint name="camera_joint_1" type="continuous">
     <parent link="base_link"/>
-    <child link="camera_link1_1"/>
+    <child link="camera_link1"/>
     <origin xyz="0.16 0.0 0.2795" rpy="0 0 0" />
     <axis xyz="0.0 0.0 -1.0" />
   </joint>
   <joint name="camera_joint_2" type="continuous">
-    <parent link="camera_link1_1"/>
-    <child link="camera_link2_1"/>
+    <parent link="camera_link1"/>
+    <child link="camera_link2"/>
     <origin xyz="0.03 0.0 0.042" rpy="0 0 0" />
     <axis xyz="0.0 1.0 0.0" />
   </joint>
   <joint name="camera_joint" type="fixed">
-    <parent link="camera_link2_1"/>
+    <parent link="camera_link2"/>
     <child link="camera_1"/>
     <origin xyz="0.020 0.01 0.015" rpy="-1.57079632679 0 -1.57079632679" />
